File: half-bridge/half-bridge.kicad_pcb (KiCad board)
At the start: 6 copper layers, 52 x 36 mm, 94 parts, among them J1 Conn_01x14, J2 MountingHole_Pad, J3 Conn_01x11_Pin, J4 Conn_01x11_Pin, J5 Conn_01x11_Pin, J6 Conn_01x11_Pin, J7 MountingHole_Pad, J8 MountingHole_Pad, J9 MountingHole_Pad, Q1 EPC2306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

Commit message: Cleanup, add more cap etc
Parts:
- added C49: 470nF, Capacitor_SMD:C_1210_3225Metric, F.Cu at (125.7, 113.3)
- added C50: 470nF, Capacitor_SMD:C_1210_3225Metric, F.Cu at (128.6, 113.3)
- added C52: 470nF, Capacitor_SMD:C_1210_3225Metric, F.Cu at (131.5, 113.3)
- added C55: 470nF, Capacitor_SMD:C_1210_3225Metric, F.Cu at (134.4, 113.3)
- added C56: 470nF, Capacitor_SMD:C_1210_3225Metric, F.Cu at (122.8, 113.3)
- added C57: 470nF, Capacitor_SMD:C_1210_3225Metric, F.Cu at (142.2, 108.8)
- added C58: 10uF, Capacitor_SMD:C_1210_3225Metric, F.Cu at (125.8, 87.6)
- added C59: 10uF, Capacitor_SMD:C_1210_3225Metric, F.Cu at (122.8, 87.6)
- added C60: 10uF, Capacitor_SMD:C_1210_3225Metric, F.Cu at (155.8, 91.5)
- C11, C15, C19, C21, C24, C26, C28, C30, C5, C7, C9: value 470nF -> 10uF
- C38, C42, C44, C45, C46, C53, C54: footprint Capacitor_SMD:C_0402_1005Metric -> Capacitor_SMD:C_0402_1005Metric_Pad0.74x0.62mm_HandSolder
- moved C43 0.50 mm to (138.1, 112.5)
- moved C41 0.20 mm to (138.1, 109.6)
Connections:
- H5 pad 1: POWER_LOW -> 0
Routing:
- net POWER_LOW: vias 50 -> 65
- net 0: vias 354 -> 365
- added copper zone on In4.Cu, net POWER_HIGH
Other:
- board text added: "Fint namn %%%date%% %%version%%"
- board text removed: "Fint namn här %%%date%% %%version%%"
