File: controller/controller.kicad_pcb (KiCad board)
At the start: 4 copper layers, 93 x 39 mm, 162 parts, among them J1 Conn_01x14, J2 Conn_01x14, J3 Conn_01x14, J4 Conn_01x14, J5 Conn_01x14, J6 USB_C_Receptacle_USB2.0_16P, J7 USB_C_Receptacle_USB2.0_16P, J8 Conn_01x03_Pin, J9 Conn_01x03_Pin, U1 STM32G474RCTx, U2 LM5168, U3 TLV76133DCY, U4 TLV76150DCY, U5 ECMF02-2AMX6, U6 ESP32-C6-WROOM-1, U7 ECMF02-2AMX6, U8 TS3011IYLT, U9 PY32F002AA15M

Commit message: More work on controller
Parts:
- removed D18, D19: BAT54S, Package_TO_SOT_SMD:SOT-23
- removed R74, R75, R76, R77, R78, R79, R80, R81, R82, R83, R84, R85, R86, R87, R88, R89, R90, R91, R92, R93: 0R, Resistor_SMD:R_0402_1005Metric
- added Q1: FDG6335N, Package_TO_SOT_SMD:SOT-363_SC-70-6, F.Cu at (107.0, 124.3)
- added Q2: FDG6335N, Package_TO_SOT_SMD:SOT-363_SC-70-6, F.Cu at (119.5, 124.3)
- added Q3: FDG6335N, Package_TO_SOT_SMD:SOT-363_SC-70-6, F.Cu at (119.5, 128.2)
- added Q4: FDG6335N, Package_TO_SOT_SMD:SOT-363_SC-70-6, F.Cu at (113.2, 124.3)
- added Q5: FDG6335N, Package_TO_SOT_SMD:SOT-363_SC-70-6, F.Cu at (113.2, 128.2)
- added Q6: FDG6335N, Package_TO_SOT_SMD:SOT-363_SC-70-6, F.Cu at (113.2, 132.2)
- added Q7: FDG6335N, Package_TO_SOT_SMD:SOT-363_SC-70-6, F.Cu at (119.5, 132.2)
- added R103: 10k, Resistor_SMD:R_0603_1608Metric, F.Cu at (106.8, 127.5)
- added R104: 10k, Resistor_SMD:R_0603_1608Metric, F.Cu at (106.8, 130.0)
- added R105: 10k, Resistor_SMD:R_0603_1608Metric, F.Cu at (106.8, 132.5)
- added R106: 10k, Resistor_SMD:R_0603_1608Metric, F.Cu at (106.8, 135.0)
- added U10: PI5C3257, Package_DFN_QFN:TQFN-16-1EP_3x3mm_P0.5mm_EP1.6x1.6mm, F.Cu at (102.2, 130.3)
- R72: value 0R -> 10k
- U8: value TS3011IYLT -> PI5C3257; footprint Package_TO_SOT_SMD:SOT-23-5 -> Package_DFN_QFN:TQFN-16-1EP_3x3mm_P0.5mm_EP1.6x1.6mm
- moved U8 50.5 mm to (102.2, 125.0)
- moved R72 35.2 mm to (101.0, 133.9)
Connections:
- D17 pad 3: COMP6_INP -> /Current_sense_4
- D20 pad 3: /Current_sense_2A -> /Current_sense_2
- D21 pad 3: /Current_sense_4 -> /Current_sense_3
- J3 pad 3: /Current_sense_3B -> unconnected-(J3-Pin_3-Pad3)
- R72 pad 1: /Current_sense_5B -> Earth
- R72 pad 2: /Current_sense_5 -> /CC_HI4_HI5_MUX
- U1 pad 10: unconnected-(U1-PC2-Pad10) -> Net-(U1-PC2)
- U1 pad 14: UCPD1_FRSTX__1 -> /NTC_3
- U1 pad 18: /Current_sense_5_ref -> ADC2_IN17
- U1 pad 19: UCPD1_FRSTX__2 -> /FRS2
- U1 pad 2: unconnected-(U1-PC13-Pad2) -> /EN_CC1
- U1 pad 20: /Current_sense_5_ref -> /FB_C
- U1 pad 22: /STM32_TX -> /NTC_5
- U1 pad 23: /STM32_RX -> /NTC_4
- U1 pad 24: /Current_sense_2A -> Net-(U1-PB0)
- U1 pad 26: Net-(U1-PB2) -> ADC2_IN12
- U1 pad 3: unconnected-(U1-PC14-Pad3) -> /EN_CC2
- U1 pad 30: unconnected-(U1-PB10-Pad30) -> HRTIM1_FLT3
- U1 pad 33: COMP6_INP -> /Current_sense_1
- U1 pad 36: Net-(D18-COM) -> /Current_sense_?
- U1 pad 37: Net-(U1-PB15) -> /PB15
- U1 pad 4: unconnected-(U1-PC15-Pad4) -> /DIR
- U1 pad 42: /HI_4 -> /PA8
- U1 pad 43: UCPD1_DBCC1 -> /PA9
- U1 pad 44: UCPD1_DBCC2 -> /PA10
- U1 pad 5: unconnected-(U1-PF0-Pad5) -> /NTC_2
- U1 pad 51: unconnected-(U1-PA15-Pad51) -> /STM32_RX
- U1 pad 52: unconnected-(U1-PC10-Pad52) -> /EN_VCONN1
- U1 pad 53: unconnected-(U1-PC11-Pad53) -> /EN_VCONN2
- U1 pad 54: unconnected-(U1-PC12-Pad54) -> /FRS1
- U1 pad 55: unconnected-(U1-PD2-Pad55) -> /CC_HI4_HI5_MUX
- U1 pad 56: UCPD1_CRS_SYNC -> /STM32_TX
- U1 pad 57: UCPD1_CC2 -> /CC2_MCU
- U1 pad 59: UCPD1_CC1 -> /CC1_MCU
- U1 pad 6: unconnected-(U1-PF1-Pad6) -> ADC2_IN10
- U1 pad 8: Net-(U1-PC0) -> /NTC_1
- U1 pad 9: Net-(U1-PC1) -> /FB_D
- U8 pad 1: HRTIM1_EEV5 -> /CC_HI4_HI5_MUX
- U8 pad 2: Earth -> unconnected-(U8-I0a-Pad2)
- U8 pad 3: /Current_sense_5 -> /HI_4
- U8 pad 4: /Current_sense_5_ref -> /PA8
- U8 pad 5: +3V3 -> /CC1_MCU
Other:
- board text added: "CS"

Commit message: Controller - More changes
Parts:
- removed Q6: FDG6335N, Package_TO_SOT_SMD:SOT-363_SC-70-6
- added D23: BAT54S, Package_TO_SOT_SMD:SOT-23, F.Cu at (87.7, 48.9)
- added D24: BAT54S, Package_TO_SOT_SMD:SOT-23, F.Cu at (101.5, 48.9)
- added D25: BAT54S, Package_TO_SOT_SMD:SOT-23, F.Cu at (108.4, 35.7)
- added D26: BAT54S, Package_TO_SOT_SMD:SOT-23, F.Cu at (101.5, 35.7)
- added D27: DFLS1200, Diode_SMD:D_PowerDI-123, F.Cu at (88.3, 25.8)
- added D28: DFLS1200, Diode_SMD:D_PowerDI-123, F.Cu at (88.3, 29.5)
- added R74: 1k, Resistor_SMD:R_0603_1608Metric, F.Cu at (93.3, 25.3)
- added R75: 1k, Resistor_SMD:R_0603_1608Metric, F.Cu at (93.3, 27.8)
- Q1, Q2, Q3, Q7: value FDG6335N -> BSS138BKS,115
- moved D22 140.3 mm to (106.7, 26.4)
- moved D17 139.7 mm to (99.8, 26.4)
- moved D16 120.9 mm to (101.5, 42.3)
- moved D15 118.5 mm to (87.7, 35.7)
- moved D20 112.7 mm to (94.6, 42.3)
- moved D13 111.7 mm to (94.6, 35.7)
- moved D21 110.8 mm to (94.6, 48.9)
- moved D14 107.7 mm to (87.7, 42.3)
- moved Q4 82.5 mm to (108.0, 41.9)
- moved Q5 82.5 mm to (108.0, 45.9)
Connections:
- D13 pad 3: /FB_A -> /FB_D
- D14 pad 3: /FB_B -> /FB_C
- D15 pad 3: /FB_C -> /FB_B
- D16 pad 3: /FB_D -> /FB_A
- D17 pad 3: /Current_sense_4 -> /Current_sense_5
- D20 pad 3: /Current_sense_2 -> /Current_sense_4
- D22 pad 3: /Current_sense_5 -> /Current_sense_2
- J6 pad A5: unconnected-(J6-CC1-PadA5) -> /CC1
- J6 pad B5: unconnected-(J6-CC2-PadB5) -> /CC2
- Q2 pad 2: /EN_CC1 -> /~{EN_CC1}
- Q2 pad 5: /EN_CC2 -> /~{EN_CC2}
- Q5 pad 1: /CC2 -> /dual_high_side_fet/OUT1
- Q5 pad 2: Net-(Q4B-D) -> Net-(Q4A-D)
- Q5 pad 3: Net-(Q5A-D) -> /dual_high_side_fet/OUT2
- Q5 pad 6: Net-(Q5A-D) -> +5V
- R105 pad 1: /EN_CC1 -> Earth
- R105 pad 2: +3V3 -> /~{EN_CC2}
- R106 pad 1: /EN_CC2 -> Earth
- R106 pad 2: +3V3 -> /~{EN_CC1}
- U1 pad 11: /FB_C -> ADC12_IN9
- U1 pad 12: /Current_sense_5 -> /NTC_5
- U1 pad 17: /Current_sense_1A -> /Current_sense_1B
- U1 pad 23: /NTC_4 -> ADC2_IN11
- U1 pad 24: Net-(U1-PB0) -> /Current_sense_1A
- U1 pad 25: /Current_sense_4 -> /Current_sense_3
- U1 pad 33: /Current_sense_1 -> /Current_sense_?
- U1 pad 36: /Current_sense_? -> /Current_sense_2
