File: controller/controller.kicad_pcb (KiCad board)
At the start: 4 copper layers, 94 x 39 mm, 170 parts, among them J1 Conn_01x14, J12 GRPB072VWQS-RC, J2 Conn_01x14, J3 Conn_01x14, J4 Conn_01x14, J5 Conn_01x14, J6 USB_C_Receptacle_USB2.0_16P, J7 USB_C_Receptacle_USB2.0_16P, J8 GRPB072VWQS-RC, J9 GRPB072VWQS-RC, U1 STM32G474RCTx, U10 PI5C3257, U11 QSBT40-7-F, U12 QSBT40-7-F, U13 QSBT40-7-F, U2 LM5169PDDAR, U3 TLV76133DCY, U4 TLV76150DCY, U5 ECMF02-2AMX6, U6 ESP32-C6-WROOM-1, U7 ECMF02-2AMX6, U8 PI5C3257, U9 PY32F002AA15M

Commit message: Controller - more changes
Parts:
- added D20: CLMUD-FKC-CHJNPM569ABB845343, Library:LED_Cree-PLCC4_1.5x1.5mm, F.Cu at (114.3, 66.0)
- added D22: LED_ARGB, Library:LED_Cree-PLCC4_1.5x1.5mm, F.Cu at (126.8, 66.0)
- added D23: CLMUD-FKC-CHJNPM569ABB845343, Library:LED_Cree-PLCC4_1.5x1.5mm, F.Cu at (139.8, 66.0)
- added D24: CLMUD-FKC-CHJNPM569ABB845343, Library:LED_Cree-PLCC4_1.5x1.5mm, F.Cu at (152.2, 66.0)
- added D25: CLMUD-FKC-CHJNPM569ABB845343, Library:LED_Cree-PLCC4_1.5x1.5mm, F.Cu at (165.2, 66.0)
- added R33: ?, Resistor_SMD:R_0402_1005Metric, F.Cu at (76.7, 117.4)
- added R34: ?, Resistor_SMD:R_0402_1005Metric, F.Cu at (76.7, 119.4)
- added R36: ?, Resistor_SMD:R_0402_1005Metric, F.Cu at (76.7, 121.4)
- added R37: ?, Resistor_SMD:R_0402_1005Metric, F.Cu at (76.7, 123.4)
- added R38: ?, Resistor_SMD:R_0402_1005Metric, F.Cu at (76.7, 125.4)
- added R40: ?, Resistor_SMD:R_0402_1005Metric, F.Cu at (76.7, 127.4)
- added R47: ?, Resistor_SMD:R_0402_1005Metric, F.Cu at (76.7, 129.4)
- added R48: ?, Resistor_SMD:R_0402_1005Metric, F.Cu at (76.7, 131.4)
- added R49: ?, Resistor_SMD:R_0402_1005Metric, F.Cu at (87.9, 117.4)
- added R50: ?, Resistor_SMD:R_0402_1005Metric, F.Cu at (87.9, 119.4)
- added R57: ?, Resistor_SMD:R_0402_1005Metric, F.Cu at (87.9, 121.4)
- added R58: ?, Resistor_SMD:R_0402_1005Metric, F.Cu at (87.9, 123.4)
- added R59: ?, Resistor_SMD:R_0402_1005Metric, F.Cu at (90.8, 117.4)
- added R60: ?, Resistor_SMD:R_0402_1005Metric, F.Cu at (90.8, 119.4)
- added R64: ?, Resistor_SMD:R_0402_1005Metric, F.Cu at (90.8, 121.4)
- added R65: ?, Resistor_SMD:R_0402_1005Metric, F.Cu at (90.8, 123.4)
- added R66: ?, Resistor_SMD:R_0402_1005Metric, F.Cu at (93.7, 117.4)
- moved C21 64.1 mm to (83.9, 85.5), turned to 180 degrees
- moved R27 63.0 mm to (83.9, 86.5), turned to 180 degrees
- moved C24 61.1 mm to (92.6, 100.1), turned to -90 degrees
- moved C22 59.9 mm to (90.4, 101.1), turned to -90 degrees
- moved R39 59.8 mm to (93.6, 100.1), turned to -90 degrees
- moved C27 58.9 mm to (88.1, 94.3), turned to 180 degrees
- moved R31 58.7 mm to (91.4, 101.1), turned to -90 degrees
- moved R82 58.1 mm to (88.1, 95.3), turned to 180 degrees
- moved C23 56.7 mm to (92.7, 96.2)
- moved R35 56.7 mm to (92.7, 95.2)
- moved U8 2.17 mm to (106.0, 89.7)
- moved R88 1.39 mm to (108.6, 96.9)
- moved R89 1.39 mm to (108.6, 95.3)
- moved R72 0.73 mm to (102.0, 88.9)
Connections:
- R10 pad 2: Net-(U6-GPIO8) -> /pwm_led7
- R7 pad 2: Net-(U6-GPIO9) -> /pwm_led4
- U6 pad 10: Net-(U6-GPIO8) -> /pwm_led7
- U6 pad 11: unconnected-(U6-GPIO10-Pad11) -> /esp32c6/IO10
- U6 pad 12: unconnected-(U6-GPIO11-Pad12) -> /esp32c6/IO11
- U6 pad 15: Net-(U6-GPIO9) -> /pwm_led4
- U6 pad 16: unconnected-(U6-GPIO18-Pad16) -> /esp32c6/IO18
- U6 pad 17: unconnected-(U6-GPIO19-Pad17) -> /esp32c6/IO19
- U6 pad 20: /STM32_TX -> /PC2
- U6 pad 21: /STM32_RX -> unconnected-(U6-GPIO23-Pad21)
- U6 pad 23: unconnected-(U6-GPIO15-Pad23) -> /esp32c6/IO15
- U6 pad 24: unconnected-(U6-U0RXD/GPIO17-Pad24) -> /STM32_TX
- U6 pad 25: unconnected-(U6-U0TXD/GPIO16-Pad25) -> /STM32_RX
- U6 pad 26: unconnected-(U6-GPIO3/ADC1_CH3-Pad26) -> /esp32c6/IO3
- U6 pad 27: unconnected-(U6-GPIO2/ADC1_CH2-Pad27) -> /esp32c6/IO2
- U6 pad 8: unconnected-(U6-GPIO0/ADC1_CH0/XTAL_32K_P-Pad8) -> /esp32c6/IO0
- U6 pad 9: unconnected-(U6-GPIO1/ADC1_CH1/XTAL_32K_N-Pad9) -> /esp32c6/IO1
Routing:
- net /LI_1: track 5.93 -> 18.2 mm
- net /HI_1: track 7.99 -> 20.1 mm
- net /LI_2: track 20.0 -> 31.2 mm
- net /HI_2: track 20.0 -> 31.1 mm
- net LI_4: track 44.9 -> 47.5 mm
