File: controller/controller.kicad_pcb (KiCad board)
At the start: 4 copper layers, 100 x 50 mm, 201 parts, among them J1 Conn_01x14, J10 Conn_ARM_JTAG_SWD_10, J11 Conn_ARM_JTAG_SWD_10, J12 GRPB072VWQS-RC, J13 GRPB072VWQS-RC, J14 Conn_01x03_Pin, J2 Conn_01x14, J3 Conn_01x14, J4 Conn_01x14, J5 Conn_01x14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

Commit message: Controller - Lots of cleanup
Parts:
- D11, D12: moved to B.Cu
- moved J14 47.2 mm to (218.3, 87.6)
- moved D12 20.9 mm to (87.5, 60.8), turned to 180 degrees
- moved D11 14.3 mm to (91.5, 60.8), turned to 0 degrees
- moved D6 13.0 mm to (140.3, 63.3), turned to -90 degrees
- moved D8 12.4 mm to (152.7, 63.3), turned to -90 degrees
- moved D10 12.3 mm to (165.3, 63.3), turned to -90 degrees
- moved D4 11.2 mm to (126.9, 63.3), turned to -90 degrees
- moved J9 4.95 mm to (104.7, 70.8)
- moved J13 4.65 mm to (104.7, 64.3), turned to -90 degrees
- moved R81 2.50 mm to (161.3, 102.7)
- moved R116 2.35 mm to (129.8, 67.5)
- moved R107 2.29 mm to (122.2, 73.2), turned to 180 degrees
- moved R74 1.79 mm to (109.2, 71.5)
- moved R114 1.70 mm to (161.7, 67.3)
- moved R112 1.55 mm to (149.7, 67.3)
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Connections:
- J12 pad 3: Earth -> /VBUS2
- J12 pad 5: /~{EN_VCONN} -> Earth
- J8 pad 4: Earth -> /VBUS1
- J8 pad 5: Earth -> /CC2
- J8 pad 6: /CC2 -> Earth
- J8 pad 7: Earth -> /CC1
- J8 pad 8: /CC1 -> /~{EN_VCONN}
Routing:
- net FB_A_FULL: track 123.0 -> 183.2 mm, vias 9 -> 14
- net /VBUS2: track 0.00 -> 19.5 mm, vias 8 -> 6
- net Net-(D19-DOUT): track 16.9 -> 0.00 mm
- net /~{EN_VCONN}: track 26.1 -> 10.7 mm
- net Logic DC/DC in: track 184.9 -> 200.1 mm, vias 13 -> 7
- net /~{EN_CC}: track 38.2 -> 23.8 mm
- net FB_D_FULL: track 150.3 -> 164.5 mm
- net /LED_CH1: track 0.00 -> 13.5 mm, vias 0 -> 1
- net /pwm_led7: track 15.1 -> 2.56 mm, vias 3 -> 0
- net /FRS: track 35.5 -> 24.3 mm
- net /VBUS1: track 0.00 -> 10.5 mm
- net +5V: track 71.1 -> 81.6 mm, vias 30 -> 32
- net /NTC_4: track 85.9 -> 96.2 mm
- net FB_B_FULL: track 148.5 -> 157.5 mm, vias 9 -> 12
- net /ESP_USB_D+: track 30.2 -> 39.0 mm
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- removed copper zone on F.Cu, net /VBUS1
- removed copper zone on In2.Cu, net /VBUS1
- removed copper zone on In1.Cu, net VBUS_A

Commit message: Controller - Some changes
Parts:
- added C41: 100nF, Capacitor_SMD:C_0402_1005Metric, F.Cu at (104.4, 82.0)
- added C42: 100nF, Capacitor_SMD:C_0402_1005Metric, F.Cu at (109.5, 82.3)
- added C43: 100nF, Capacitor_SMD:C_0402_1005Metric, B.Cu at (124.7, 79.7)
- added C44: 100nF, Capacitor_SMD:C_0402_1005Metric, B.Cu at (135.7, 80.2)
- added C45: 100nF, Capacitor_SMD:C_0402_1005Metric, F.Cu at (149.1, 79.9)
- added C61: 100nF, Capacitor_SMD:C_0402_1005Metric, F.Cu at (161.6, 80.7)
- added C62: 100nF, Capacitor_SMD:C_0402_1005Metric, F.Cu at (167.0, 83.0)
- added Q1: BSS138, Package_TO_SOT_SMD:SOT-23, B.Cu at (89.5, 83.6)
- added Q2: BSS138, Package_TO_SOT_SMD:SOT-23, F.Cu at (99.2, 119.9)
- added R25: ?k, Resistor_SMD:R_0402_1005Metric, F.Cu at (98.2, 123.1)
- added R26: ?k, Resistor_SMD:R_0402_1005Metric, F.Cu at (98.2, 125.1)
- moved J12 5.00 mm to (83.0, 70.3), turned to 180 degrees
- moved J8 5.00 mm to (96.2, 70.3), turned to 180 degrees
Connections:
- J12 pad 7: /CC2_MCU -> /OTHER_USB_CC2
- J12 pad 9: /CC1_MCU -> /OTHER_USB_CC1
- J9 pad 6: /OTHER_USB_CC2 -> unconnected-(J9-Pin_6-Pad6)
- J9 pad 8: /OTHER_USB_CC1 -> unconnected-(J9-Pin_8-Pad8)
- R10 pad 2: /LED_CH1 -> /esp32c6/LED_CH1
- U6 pad 10: /LED_CH1 -> /esp32c6/LED_CH1
- U6 pad 20: /LED_CH2 -> /esp32c6/LED_CH2
Routing:
- net /CC2_MCU: track 49.3 -> 39.8 mm
- net /OTHER_USB_CC1: track 0.00 -> 7.23 mm
- net /CC1: track 0.00 -> 5.78 mm, vias 0 -> 1
- net /CC1_MCU: track 52.1 -> 48.1 mm, vias 4 -> 3
- net /CC2: track 0.00 -> 3.61 mm, vias 0 -> 1
- net /LED_CH1: track 13.5 -> 9.91 mm
- net Earth: track 17.7 -> 20.7 mm, vias 160 -> 174
- net /esp32c6/LED_CH1: track 0.00 -> 1.80 mm
- net +5V: track 81.6 -> 83.0 mm
- net /NTC_4: track 96.2 -> 96.8 mm
- net /VBUS1: vias 8 -> 4
- net +3V3: vias 18 -> 17

Commit message: Controller - Some changes
Parts:
- added C63: 100nF, Capacitor_SMD:C_0402_1005Metric, B.Cu at (97.9, 84.5)
- moved R75 3.16 mm to (110.2, 98.1)
- moved R87 2.83 mm to (110.2, 101.9)
- moved R86 2.65 mm to (110.2, 100.0)
- moved R89 1.00 mm to (110.2, 105.7)
- moved R88 0.78 mm to (110.2, 103.8)
- moved R74 0.40 mm to (108.8, 71.5)
Connections:
- J9 pad 6: unconnected-(J9-Pin_6-Pad6) -> /CC2_MCU
- J9 pad 8: unconnected-(J9-Pin_8-Pad8) -> /CC1_MCU
Routing:
- net FB_D_FULL: track 164.5 -> 206.8 mm, vias 13 -> 15
- net FB_C_FULL: track 169.5 -> 196.7 mm, vias 14 -> 15
- net FB_B_FULL: track 157.5 -> 181.7 mm, vias 12 -> 11
- net FB_A_FULL: track 183.2 -> 205.4 mm, vias 14 -> 15
- net /LED_CH1: track 9.91 -> 24.6 mm, vias 1 -> 4
- net /CC2: track 3.61 -> 16.5 mm
- net +3V3: track 43.0 -> 55.1 mm
- net /NTC_4: track 96.8 -> 104.6 mm, vias 4 -> 6
- net /VBUS1: track 10.5 -> 14.5 mm, vias 4 -> 5
- net /hb-card3/Current_sense: track 56.8 -> 53.0 mm
- net /PA5: track 24.6 -> 28.1 mm
- net /hb-card2/Current_sense: track 46.7 -> 43.8 mm
- net /hb-card1/Current_sense: track 36.6 -> 34.4 mm
- net /CC_HI4_HI5_MUX: track 30.3 -> 32.4 mm
- net /CC_SELECT: track 27.9 -> 29.8 mm
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
Commit message: Controller - More routing
Connections:
- J8 pad 10: 6-18V -> +3V3
- J8 pad 3: Earth -> /VBUS1
- J8 pad 4: /VBUS1 -> Earth
- J8 pad 9: +3V3 -> 6-18V
Routing:
- net 6-18V: track 17.8 -> 45.0 mm, vias 10 -> 15
- net +3V3: track 55.1 -> 78.8 mm, vias 17 -> 16
- net /CC1_MCU: track 48.1 -> 33.7 mm
- net /OTHER_USB_CC2: track 0.00 -> 10.2 mm, vias 0 -> 1
- net /CC_SELECT: track 29.8 -> 20.9 mm
- net /CC2_MCU: track 38.9 -> 30.7 mm, vias 3 -> 2
- net /CC2: track 16.5 -> 10.7 mm
- net /OTHER_USB_CC1: track 7.23 -> 5.55 mm
- net /FRS: track 24.3 -> 22.9 mm, vias 3 -> 1
- net Earth: track 20.4 -> 21.9 mm, vias 174 -> 175
- net /NTC_4: track 104.6 -> 103.4 mm
- net /LED_CH1: track 24.6 -> 23.7 mm, vias 4 -> 3
- net Net-(D14-DOUT): track 8.82 -> 9.59 mm
- net /~{EN_CC}: track 24.5 -> 25.1 mm
- net FB_C_FULL: track 196.7 -> 197.3 mm
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- added copper zone on F.Cu, net /VBUS1
- added copper zone on In2.Cu, net /VBUS1
