File: controller/dual_high_side_fet.kicad_sch (KiCad schematic)
At the start: 5 parts, among them Q2 BSS138BKS,115, Q3 BSS138BKS,115, Q7 BSS138BKS,115

Commit message: Controller - More changes
Parts:
- removed Q2, Q3, Q7: BSS138BKS,115, Package_TO_SOT_SMD:SOT-363_SC-70-6, symbol Transistor_FET:FDG6335N
- removed R101, R99: 10k, symbol Device:R
- added Q4: BSS138BKS,115, Package_TO_SOT_SMD:SOT-363_SC-70-6, symbol Transistor_FET:FDG6335N
- added Q5: FDG6335N, Package_TO_SOT_SMD:SOT-363_SC-70-6, symbol Transistor_FET:FDG6335N
- added R76, R77: 10k, symbol Device:R
Connections:
- net 6-18V: now also R76.1, R77.1
- net Earth: now also Q4.1 (S), Q4.4 (S)
- net IN1: now also Q5.6 (D)
- net IN2: now also Q5.4 (S)
- new net: Q4.3 (D), Q5.5 (G), R77.2
- new net: Q4.6 (D), Q5.2 (G), R76.2
- new net OUT1: Q5.1 (S)
- new net OUT2: Q5.3 (D)
- new net ~{EN1}: Q4.2 (G)
- new net ~{EN2}: Q4.5 (G)
