File: controller/mcu_clamp.kicad_sch (KiCad schematic)
At the start: 1 part

Commit message: Controller - Try to simplify
Parts:
- renumbered D17 to D26
Changed lines of the file:
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@@
 		(dnp no)
 		(fields_autoplaced yes)
-		(property "Reference" "D17"
+		(property "Reference" "D26"
 			(at 60.96 62.2299 90)
 			(effects
@@
 		(instances
 			(project "controller"
-				(path "/5b092a03-7e3e-4df1-ad91-2ac0e362f857/2daf64ca-0fcc-4c79-982b-99a1ed63087f"
-					(reference "D17")
-					(unit 1)
-				)
-				(path "/5b092a03-7e3e-4df1-ad91-2ac0e362f857/3e515984-b506-4b34-9c6c-a071ff059aee"
-					(reference "D22")
-					(unit 1)
-				)
-				(path "/5b092a03-7e3e-4df1-ad91-2ac0e362f857/6d8a5e30-be0a-415d-800e-7055fa910833"
-					(reference "D20")
-					(unit 1)
-				)
-				(path "/5b092a03-7e3e-4df1-ad91-2ac0e362f857/8b708188-1a68-474c-8138-666e57805904"
-					(reference "D21")
-					(unit 1)
-				)
 				(path "/5b092a03-7e3e-4df1-ad91-2ac0e362f857/bfb44169-033d-4821-bbb7-0e04a8e5768b"
 					(reference "D26")
@@
 				(path "/5b092a03-7e3e-4df1-ad91-2ac0e362f857/e36b8f0b-f67b-43b4-a062-1c2e4f599a7e"
 					(reference "D25")
-					(unit 1)
-				)
-				(path "/5b092a03-7e3e-4df1-ad91-2ac0e362f857/2f911ebd-6dc8-4496-8afb-4a9ec6bafab7/17fa42ce-3bca-4df7-8e9c-f893032f2f24"
-					(reference "D15")
-					(unit 1)
-				)
-				(path "/5b092a03-7e3e-4df1-ad91-2ac0e362f857/3a11ce7c-7e29-4758-a12a-8535ab4c73af/17fa42ce-3bca-4df7-8e9c-f893032f2f24"
-					(reference "D18")
-					(unit 1)
-				)
-				(path "/5b092a03-7e3e-4df1-ad91-2ac0e362f857/8b76543b-a49c-413b-a98c-7f3e228c6216/17fa42ce-3bca-4df7-8e9c-f893032f2f24"
-					(reference "D13")
-					(unit 1)
-				)
-				(path "/5b092a03-7e3e-4df1-ad91-2ac0e362f857/a5d84eb1-8829-4f32-a763-e01f5977372c/17fa42ce-3bca-4df7-8e9c-f893032f2f24"
-					(reference "D14")
-					(unit 1)
-				)
-				(path "/5b092a03-7e3e-4df1-ad91-2ac0e362f857/dfe157ff-eae8-44d0-adc3-b7fe75c1e740/17fa42ce-3bca-4df7-8e9c-f893032f2f24"
-					(reference "D16")
-					(unit 1)
-				)
-				(path "/5b092a03-7e3e-4df1-ad91-2ac0e362f857/e3d09b0d-badf-46a0-b7fb-f25da99c9c12/17fa42ce-3bca-4df7-8e9c-f893032f2f24"
-					(reference "D19")
 					(unit 1)
 				)
@@
 		(dnp no)
 		(fields_autoplaced yes)
-		(property "Reference" "#PWR092"
+		(property "Reference" "#PWR0117"
 			(at 63.5 59.69 0)
 			(effects
@@
 		(instances
 			(project "controller"
-				(path "/5b092a03-7e3e-4df1-ad91-2ac0e362f857/2daf64ca-0fcc-4c79-982b-99a1ed63087f"
-					(reference "#PWR092")
-					(unit 1)
-				)
-				(path "/5b092a03-7e3e-4df1-ad91-2ac0e362f857/3e515984-b506-4b34-9c6c-a071ff059aee"
-					(reference "#PWR0114")
-					(unit 1)
-				)
-				(path "/5b092a03-7e3e-4df1-ad91-2ac0e362f857/6d8a5e30-be0a-415d-800e-7055fa910833"
-					(reference "#PWR0110")
-					(unit 1)
-				)
-				(path "/5b092a03-7e3e-4df1-ad91-2ac0e362f857/8b708188-1a68-474c-8138-666e57805904"
-					(reference "#PWR0112")
-					(unit 1)
-				)
 				(path "/5b092a03-7e3e-4df1-ad91-2ac0e362f857/bfb44169-033d-4821-bbb7-0e04a8e5768b"
 					(reference "#PWR0117")
@@
 				(path "/5b092a03-7e3e-4df1-ad91-2ac0e362f857/e36b8f0b-f67b-43b4-a062-1c2e4f599a7e"
 					(reference "#PWR0108")
-					(unit 1)
-				)
-				(path "/5b092a03-7e3e-4df1-ad91-2ac0e362f857/2f911ebd-6dc8-4496-8afb-4a9ec6bafab7/17fa42ce-3bca-4df7-8e9c-f893032f2f24"
-					(reference "#PWR077")
-					(unit 1)
-				)
-				(path "/5b092a03-7e3e-4df1-ad91-2ac0e362f857/3a11ce7c-7e29-4758-a12a-8535ab4c73af/17fa42ce-3bca-4df7-8e9c-f893032f2f24"
-					(reference "#PWR088")
-					(unit 1)
-				)
-				(path "/5b092a03-7e3e-4df1-ad91-2ac0e362f857/8b76543b-a49c-413b-a98c-7f3e228c6216/17fa42ce-3bca-4df7-8e9c-f893032f2f24"
-					(reference "#PWR040")
-					(unit 1)
-				)
-				(path "/5b092a03-7e3e-4df1-ad91-2ac0e362f857/a5d84eb1-8829-4f32-a763-e01f5977372c/17fa42ce-3bca-4df7-8e9c-f893032f2f24"
-					(reference "#PWR051")
-					(unit 1)
-				)
-				(path "/5b092a03-7e3e-4df1-ad91-2ac0e362f857/dfe157ff-eae8-44d0-adc3-b7fe75c1e740/17fa42ce-3bca-4df7-8e9c-f893032f2f24"
-					(reference "#PWR080")
-					(unit 1)
-				)
-				(path "/5b092a03-7e3e-4df1-ad91-2ac0e362f857/e3d09b0d-badf-46a0-b7fb-f25da99c9c12/17fa42ce-3bca-4df7-8e9c-f893032f2f24"
-					(reference "#PWR0100")
 					(unit 1)
 				)
@@
 		(dnp no)
 		(fields_autoplaced yes)
-		(property "Reference" "#PWR093"
+		(property "Reference" "#PWR0118"
 			(at 63.5 77.47 0)
 			(effects
@@
 		(instances
 			(project "controller"
-				(path "/5b092a03-7e3e-4df1-ad91-2ac0e362f857/2daf64ca-0fcc-4c79-982b-99a1ed63087f"
-					(reference "#PWR093")
-					(unit 1)
-				)
-				(path "/5b092a03-7e3e-4df1-ad91-2ac0e362f857/3e515984-b506-4b34-9c6c-a071ff059aee"
-					(reference "#PWR0115")
-					(unit 1)
-				)
-				(path "/5b092a03-7e3e-4df1-ad91-2ac0e362f857/6d8a5e30-be0a-415d-800e-7055fa910833"
-					(reference "#PWR0111")
-					(unit 1)
-				)
-				(path "/5b092a03-7e3e-4df1-ad91-2ac0e362f857/8b708188-1a68-474c-8138-666e57805904"
-					(reference "#PWR0113")
-					(unit 1)
-				)
 				(path "/5b092a03-7e3e-4df1-ad91-2ac0e362f857/bfb44169-033d-4821-bbb7-0e04a8e5768b"
 					(reference "#PWR0118")
@@
 					(unit 1)
 				)
-				(path "/5b092a03-7e3e-4df1-ad91-2ac0e362f857/2f911ebd-6dc8-4496-8afb-4a9ec6bafab7/17fa42ce-3bca-4df7-8e9c-f893032f2f24"
-					(reference "#PWR078")
-					(unit 1)
-				)
-				(path "/5b092a03-7e3e-4df1-ad91-2ac0e362f857/3a11ce7c-7e29-4758-a12a-8535ab4c73af/17fa42ce-3bca-4df7-8e9c-f893032f2f24"
-					(reference "#PWR089")
-					(unit 1)
-				)
-				(path "/5b092a03-7e3e-4df1-ad91-2ac0e362f857/8b76543b-a49c-413b-a98c-7f3e228c6216/17fa42ce-3bca-4df7-8e9c-f893032f2f24"
-					(reference "#PWR047")
-					(unit 1)
-				)
-				(path "/5b092a03-7e3e-4df1-ad91-2ac0e362f857/a5d84eb1-8829-4f32-a763-e01f5977372c/17fa42ce-3bca-4df7-8e9c-f893032f2f24"
-					(reference "#PWR052")
-					(unit 1)
-				)
-				(path "/5b092a03-7e3e-4df1-ad91-2ac0e362f857/dfe157ff-eae8-44d0-adc3-b7fe75c1e740/17fa42ce-3bca-4df7-8e9c-f893032f2f24"
-					(reference "#PWR081")
-					(unit 1)
-				)
-				(path "/5b092a03-7e3e-4df1-ad91-2ac0e362f857/e3d09b0d-badf-46a0-b7fb-f25da99c9c12/17fa42ce-3bca-4df7-8e9c-f893032f2f24"
-					(reference "#PWR0101")
-					(unit 1)
-				)
