File: controller/controller.kicad_sch (KiCad schematic)
At the start: 96 parts, among them J11 Conn_ARM_JTAG_SWD_10, J12 GRPB072VWQS-RC, J13 GRPB072VWQS-RC, J6 USB_C_Receptacle_USB2.0_16P, J7 USB_C_Receptacle_USB2.0_16P, J8 GRPB072VWQS-RC, J9 GRPB072VWQS-RC, SW3 Boot, SW4 Reset, SW5 SW_Nidec_CAS-120A1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

Commit message: Controller - More routing
Parts:
- C7, C8: value 4.7uF -> 10uF
Connections:
- net Current_sense_1A is gone; now on net Current_sense_1: U9.5 (Pin_5)
Changed lines of the file:
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@@
 		)
 	)
-	(label "Current_sense_1A"
+	(label "Current_sense_1"
 		(at 30.48 71.12 0)
 		(fields_autoplaced yes)
@@
 			)
 		)
-		(property "Value" "4.7uF"
+		(property "Value" "10uF"
 			(at 373.38 290.8362 0)
 			(effects
@@
 			)
 		)
-		(property "Value" "4.7uF"
+		(property "Value" "10uF"
 			(at 373.38 271.7862 0)
 			(effects

Commit message: Controller - More routing
Connections:
- net Current_sense_2B is gone; now on net Current_sense_2: R29.2
Changed lines of the file:
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@@
 		)
 	)
-	(label "Current_sense_2B"
+	(label "Current_sense_2"
 		(at 209.55 52.07 180)
 		(fields_autoplaced yes)

Commit message: Controller - Expand to 100x40mm
Parts:
- removed U11: QSBT40-7-F, Package_TO_SOT_SMD:SOT-363_SC-70-6, symbol Library:QSBT40-7-F
Connections:
- net Current_sense_1: no longer U14.4 (DL2)
Other:
- moved on the sheet: U14B, U14C

Commit message: Add new led
Parts:
- removed R29: 0R, Resistor_SMD:R_0402_1005Metric, symbol Device:R_Small
- added D26: WS2812B, LED_SMD:LED_WS2812_PLCC6_5.0x5.0mm_P1.6mm, symbol LED:WS2812B
Changed lines of the file:
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@@
 	(wire
 		(pts
-			(xy 191.77 52.07) (xy 209.55 52.07)
-		)
-		(stroke
-			(width 0)
-			(type default)
-		)
-	)
-	(wire
-		(pts
 			(xy 170.18 34.29) (xy 176.53 34.29)
 		)
@@
 	(wire
 		(pts
-			(xy 167.64 52.07) (xy 186.69 52.07)
+			(xy 167.64 52.07) (xy 185.42 52.07)
 		)
 		(stroke
@@
 		)
 	)
-	(label "Current_sense_2"
-		(at 209.55 52.07 180)
-		(fields_autoplaced yes)
-		(effects
-			(font
-				(size 1.27 1.27)
-			)
-			(justify right bottom)
-		)
-	)
 	(label "CC_HI4_HI5_MUX"
 		(at 269.24 187.96 0)
@@
 	)
 	(symbol
+		(lib_id "LED:WS2812B")
+		(at 387.35 219.71 0)
+		(unit 1)
+		(exclude_from_sim no)
+		(in_bom yes)
+		(on_board yes)
+		(dnp no)
+		(fields_autoplaced yes)
+		(property "Reference" "D26"
+			(at 398.78 213.3914 0)
+			(effects
+				(font
+					(size 1.27 1.27)
+				)
+			)
+		)
+		(property "Value" "WS2812B"
+			(at 398.78 215.9314 0)
+			(effects
+				(font
+					(size 1.27 1.27)
+				)
+			)
+		)
+		(property "Footprint" "LED_SMD:LED_WS2812_PLCC6_5.0x5.0mm_P1.6mm"
+			(at 388.62 227.33 0)
+			(effects
+				(font
+					(size 1.27 1.27)
+				)
+				(justify left top)
+				(hide yes)
+			)
+		)
+		(property "Datasheet" "https://cdn-shop.adafruit.com/datasheets/WS2812B.pdf"
+			(at 389.89 229.235 0)
+			(effects
+				(font
+					(size 1.27 1.27)
+				)
+				(justify left top)
+				(hide yes)
+			)
+		)
+		(property "Description" "RGB LED with integrated controller"
+			(at 387.35 219.71 0)
+			(effects
+				(font
+					(size 1.27 1.27)
+				)
+				(hide yes)
+			)
+		)
+		(pin "4"
+		)
+		(pin "1"
+		)
+		(pin "3"
+		)
+		(pin "2"
+		)
+		(instances
+			(project ""
+				(path "/5b092a03-7e3e-4df1-ad91-2ac0e362f857"
+					(reference "D26")
+					(unit 1)
+				)
+			)
+		)
+	)
+	(symbol
 		(lib_id "Switch:SW_Push")
 		(at 227.33 113.03 0)
@@
 					(unit 1)
 				)
-			)
-		)
-	)
-	(symbol
-		(lib_id "Device:R_Small")
-		(at 189.23 52.07 90)
-		(unit 1)
-		(exclude_from_sim no)
-		(in_bom yes)
-		(on_board yes)
-		(dnp no)
-		(fields_autoplaced yes)
-		(property "Reference" "R29"
-			(at 189.23 46.99 90)
-			(effects
-				(font
-					(size 1.27 1.27)
-				)
-			)
-		)
-		(property "Value" "0R"
-			(at 189.23 49.53 90)
-			(effects
-				(font
-					(size 1.27 1.27)
-				)
-			)
-		)
-		(property "Footprint" "Resistor_SMD:R_0402_1005Metric"
-			(at 189.23 52.07 0)
-			(effects
-				(font
-					(size 1.27 1.27)
-				)
-				(hide yes)
-			)
-		)
-		(property "Datasheet" "~"
-			(at 189.23 52.07 0)
-			(effects
-				(font
-					(size 1.27 1.27)
-				)
-				(hide yes)
-			)
-		)
-		(property "Description" "Resistor, small symbol"
-			(at 189.23 52.07 0)
-			(effects
-				(font
-					(size 1.27 1.27)
-				)
-				(hide yes)
-			)
-		)
-		(pin "1"
-		)
-		(pin "2"
-		)
-		(instances
-			(project "controller"
-				(path "/5b092a03-7e3e-4df1-ad91-2ac0e362f857"
-					(reference "R29")
-					(unit 1)
-				)

Commit message: Add new leds
Parts:
- removed D13, D14, D15, D16, D17, D18, D19, D21: LED, symbol Device:LED
- removed D20: CLMUD-FKC-CHJNPM569ABB845343, Library:LED_Cree-PLCC4_1.5x1.5mm, symbol Device:LED_ARGB
- removed D22: LED_ARGB, Library:LED_Cree-PLCC4_1.5x1.5mm, symbol Device:LED_ARGB
- removed D26: WS2812B, LED_SMD:LED_WS2812_PLCC6_5.0x5.0mm_P1.6mm, symbol LED:WS2812B
- removed R25, R26: 0R, Resistor_SMD:R_0402_1005Metric, symbol Device:R_Small
- removed R33, R34, R36, R37, R38, R40, R47, R48: ?, Resistor_SMD:R_0402_1005Metric, symbol Device:R_Small
- added D13, D14, D15, D16, D17, D18, D19: WS2812B, LED_SMD:LED_WS2812B_PLCC4_5.0x5.0mm_P3.2mm, symbol LED:WS2812B
- added J14: Conn_01x03_Pin, Connector_PinHeader_2.54mm:PinHeader_1x03_P2.54mm_Vertical, symbol Connector:Conn_01x03_Pin
Connections:
- net +5V: now also D13.1 (VDD), D14.1 (VDD), D15.1 (VDD), D16.1 (VDD), D17.1 (VDD), D18.1 (VDD), D19.1 (VDD), J14.3 (Pin_3)
- net Earth: now also D13.3 (VSS), D14.3 (VSS), D15.3 (VSS), D16.3 (VSS), D17.3 (VSS), D18.3 (VSS), D19.3 (VSS), J14.2 (Pin_2)
- new net: D18.2 (DOUT), D19.4 (DIN)
- new net: D17.2 (DOUT), D18.4 (DIN)
- new net: D19.2 (DOUT), J14.1 (Pin_1)
- new net: D16.2 (DOUT), D17.4 (DIN)
- new net: D15.2 (DOUT), D16.4 (DIN)
- new net: D14.2 (DOUT), D15.4 (DIN)
- new net: D13.2 (DOUT), D14.4 (DIN)
- new net LED_CH1: D13.4 (DIN)
Other:
- sheet esp32c6 ports: added LED_CH1, LED_CH2; removed G, R

Commit message: Controller - Expand to 100x50mm to allow VBUS to go around
Parts:
- C1: footprint Capacitor_SMD:C_1210_3225Metric -> Capacitor_SMD:C_1206_3216Metric
- J14: footprint Connector_PinHeader_2.54mm:PinHeader_1x03_P2.54mm_Vertical -> Connector_PinHeader_2.54mm:PinHeader_1x03_P2.54mm_Vertical_SMD_Pin1Left
Changed lines of the file:
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@@
 			)
 		)
-		(property "Footprint" "Connector_PinHeader_2.54mm:PinHeader_1x03_P2.54mm_Vertical"
+		(property "Footprint" "Connector_PinHeader_2.54mm:PinHeader_1x03_P2.54mm_Vertical_SMD_Pin1Left"
 			(at 538.48 165.1 0)
 			(effects
@@
 			)
 		)
-		(property "Footprint" "Capacitor_SMD:C_1210_3225Metric"
+		(property "Footprint" "Capacitor_SMD:C_1206_3216Metric"
 			(at 227.33 273.05 0)
 			(effects

Commit message: Controller - Lots of cleanup
Connections:
- net CC1: now also J8.7 (Pin_7); no longer J8.8 (Pin_8)
- net CC2: now also J8.5 (Pin_5); no longer J8.6 (Pin_6)
- net Earth: now also J12.5 (Pin_5), J8.6 (Pin_6); no longer J12.3 (Pin_3), J8.4 (Pin_4), J8.5 (Pin_5), J8.7 (Pin_7)
- net VBUS1: now also J8.4 (Pin_4)
- net VBUS2: now also J12.3 (Pin_3)
- net ~{EN_VCONN}: now also J8.8 (Pin_8); no longer J12.5 (Pin_5)
Changed lines of the file:
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@@
 	)
 	(junction
-		(at 76.2 320.04)
-		(diameter 0)
-		(color 0 0 0 0)
-	)
-	(junction
 		(at 236.22 270.51)
 		(diameter 0)
@@
 	)
 	(junction
-		(at 76.2 322.58)
-		(diameter 0)
-		(color 0 0 0 0)
-	)
-	(junction
 		(at 60.96 57.15)
 		(diameter 0)
@@
 	)
 	(junction
+		(at 76.2 298.45)
+		(diameter 0)
+		(color 0 0 0 0)
+	)
+	(junction
 		(at 176.53 34.29)
 		(diameter 0)
@@
 	)
 	(junction
+		(at 63.5 325.12)
+		(diameter 0)
+		(color 0 0 0 0)
+	)
+	(junction
 		(at 149.86 44.45)
 		(diameter 0)
@@
 	(wire
 		(pts
+			(xy 63.5 322.58) (xy 63.5 325.12)
+		)
+		(stroke
+			(width 0)
+			(type default)
+		)
+	)
+	(wire
+		(pts
 			(xy 236.22 270.51) (xy 236.22 275.59)
 		)
@@
 	(wire
 		(pts
-			(xy 63.5 314.96) (xy 55.88 314.96)
+			(xy 63.5 314.96) (xy 50.8 314.96)
 		)
 		(stroke
@@
 	(wire
 		(pts
-			(xy 76.2 322.58) (xy 83.82 322.58)
+			(xy 63.5 320.04) (xy 55.88 320.04)
 		)
 		(stroke
@@
 	(wire
 		(pts
-			(xy 60.96 317.5) (xy 63.5 317.5)
+			(xy 78.74 317.5) (xy 76.2 317.5)
 		)
 		(stroke
@@
 	(wire
 		(pts
-			(xy 87.63 293.37) (xy 76.2 293.37)
+			(xy 52.07 317.5) (xy 63.5 317.5)
 		)
 		(stroke
@@
 	(wire
 		(pts
-			(xy 76.2 320.04) (xy 76.2 322.58)
-		)
-		(stroke
-			(width 0)
-			(type default)
-		)
-	)
-	(wire
-		(pts
 			(xy 398.78 22.86) (xy 405.13 22.86)
 		)
@@
 	(wire
 		(pts
-			(xy 60.96 320.04) (xy 63.5 320.04)
+			(xy 78.74 320.04) (xy 76.2 320.04)
 		)
 		(stroke
@@
 	(wire
 		(pts
-			(xy 76.2 317.5) (xy 76.2 320.04)
-		)
-		(stroke
-			(width 0)
-			(type default)
-		)
-	)
-	(wire
-		(pts
 			(xy 104.14 237.49) (xy 104.14 236.22)
 		)
@@
 	(wire
 		(pts
-			(xy 60.96 322.58) (xy 63.5 322.58)
+			(xy 76.2 295.91) (xy 76.2 298.45)
+		)
+		(stroke
+			(width 0)
+			(type default)
+		)
+	)
+	(wire
+		(pts
+			(xy 78.74 322.58) (xy 76.2 322.58)
 		)
 		(stroke
@@
 	(wire
 		(pts
-			(xy 76.2 295.91) (xy 85.09 295.91)
+			(xy 76.2 293.37) (xy 85.09 293.37)
 		)
 		(stroke
@@
 	)
 	(label "~{EN_VCONN}"
-		(at 87.63 293.37 180)
+		(at 52.07 317.5 0)
 		(fields_autoplaced yes)
 		(effects
@@
 				(size 1.27 1.27)
 			)
-			(justify right bottom)
+			(justify left bottom)
 		)
 	)
@@
 	)
 	(label "CC1"
-		(at 60.96 317.5 180)
+		(at 78.74 317.5 0)
 		(fields_autoplaced yes)
 		(effects
@@
 				(size 1.27 1.27)
 			)
-			(justify right bottom)
+			(justify left bottom)
 		)
 	)
@@
 	)
 	(label "CC2"
-		(at 60.96 320.04 180)
+		(at 78.74 320.04 0)
 		(fields_autoplaced yes)
 		(effects
@@
 				(size 1.27 1.27)
 			)
-			(justify right bottom)
+			(justify left bottom)
 		)
 	)
@@
 	(global_label "6-18V"
 		(shape input)
-		(at 55.88 314.96 180)
+		(at 50.8 314.96 180)
 		(fields_autoplaced yes)
 		(effects
@@
 		)
 		(property "Intersheetrefs" "${INTERSHEET_REFS}"
-			(at 46.6053 314.96 0)
+			(at 41.5253 314.96 0)
 			(effects
 				(font
@@
 	(symbol
 		(lib_id "power:Earth")
-		(at 60.96 322.58 0)
+		(at 78.74 322.58 0)
+		(mirror y)
 		(unit 1)
 		(exclude_from_sim no)
@@
 		(fields_autoplaced yes)
 		(property "Reference" "#PWR086"
-			(at 60.96 328.93 0)
+			(at 78.74 328.93 0)
 			(effects
 				(font
@@
 		)
 		(property "Value" "Earth"
-			(at 60.96 326.39 0)
+			(at 78.74 326.39 0)
 			(effects
 				(font
@@
 		)
 		(property "Footprint" ""
-			(at 60.96 322.58 0)
+			(at 78.74 322.58 0)
 			(effects
 				(font
@@
 		)
 		(property "Datasheet" "~"
-			(at 60.96 322.58 0)
+			(at 78.74 322.58 0)
 			(effects
 				(font
@@
 		)
 		(property "Description" ""
-			(at 60.96 322.58 0)
+			(at 78.74 322.58 0)
 			(effects
 				(font
@@
 	(symbol
 		(lib_id "power:Earth")
-		(at 83.82 322.58 0)
+		(at 55.88 320.04 0)
+		(mirror y)
 		(unit 1)
 		(exclude_from_sim no)
@@
 		(fields_autoplaced yes)
 		(property "Reference" "#PWR0123"
-			(at 83.82 328.93 0)
+			(at 55.88 326.39 0)
 			(effects
 				(font
@@
 		)
 		(property "Value" "Earth"
-			(at 83.82 326.39 0)
+			(at 55.88 323.85 0)
 			(effects
 				(font
@@
 		)
 		(property "Footprint" ""
-			(at 83.82 322.58 0)
+			(at 55.88 320.04 0)
 			(effects
 				(font
@@
 		)
 		(property "Datasheet" "~"
-			(at 83.82 322.58 0)
+			(at 55.88 320.04 0)
 			(effects
 				(font
@@
 		)
 		(property "Description" ""
-			(at 83.82 322.58 0)
+			(at 55.88 320.04 0)
 			(effects
 				(font
@@
 	(symbol
 		(lib_id "power:Earth")
-		(at 85.09 295.91 0)
+		(at 85.09 293.37 0)
 		(unit 1)
 		(exclude_from_sim no)
@@
 		(fields_autoplaced yes)
 		(property "Reference" "#PWR063"
-			(at 85.09 302.26 0)
+			(at 85.09 299.72 0)
 			(effects
 				(font
@@
 		)
 		(property "Value" "Earth"
-			(at 85.09 299.72 0)
+			(at 85.09 297.18 0)
 			(effects
 				(font
@@
 		)
 		(property "Footprint" ""
-			(at 85.09 295.91 0)
+			(at 85.09 293.37 0)
 			(effects
 				(font
@@
 		)
 		(property "Datasheet" "~"
-			(at 85.09 295.91 0)
+			(at 85.09 293.37 0)
 			(effects
 				(font
@@
 		)
 		(property "Description" ""
-			(at 85.09 295.91 0)
+			(at 85.09 293.37 0)
 			(effects
 				(font
