File: controller/esp32c6.kicad_sch (KiCad schematic)
At the start: 12 parts, among them J10 Conn_ARM_JTAG_SWD_10, SW1 Boot, SW2 Reset, U6 ESP32-C6-WROOM-1

Commit message: controller - Update BOM
Parts:
- C15, C20: ARTIKELKOD (none) -> 065-00248
- C16, C17, C18: ARTIKELKOD (none) -> 065-00195
- J10: ARTIKELKOD (none) -> ?
- R11: ARTIKELKOD (none) -> 035-00451 (15k)
- R12: ARTIKELKOD (none) -> 035-00209
- R7: ARTIKELKOD (none) -> 035-00134
- SW1, SW2: ARTIKELKOD (none) -> -; MFR (none) -> Omron Electronics Inc-EMC Div; part-num (none) -> B3U-1000P
- U6: ARTIKELKOD (none) -> -; MFR (none) -> Espressif Systems; part-num (none) -> ESP32-C6-WROOM-1
Changed lines of the file:
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@@
+			)
+		)
+		(property "ARTIKELKOD" "065-00195"
+			(at 151.13 63.5 0)
+			(effects
+				(font
+					(size 1.27 1.27)
+				)
+				(hide yes)
 			)
 		)
@@
 			)
 		)
+		(property "ARTIKELKOD" "035-00134"
+			(at 90.17 91.44 0)
+			(effects
+				(font
+					(size 1.27 1.27)
+				)
+				(hide yes)
+			)
+		)
 		(pin "1"
 		)
@@
 			)
 		)
+		(property "ARTIKELKOD" "065-00195"
+			(at 156.21 63.5 0)
+			(effects
+				(font
+					(size 1.27 1.27)
+				)
+				(hide yes)
+			)
+		)
 		(pin "2"
 		)
@@
 			)
 		)
-		(property "MFR" ""
+		(property "MFR" "Espressif Systems"
 			(at 128.27 101.6 0)
 			(effects
@@
 			)
 		)
-		(property "part-num" ""
+		(property "part-num" "ESP32-C6-WROOM-1"
+			(at 128.27 101.6 0)
+			(effects
+				(font
+					(size 1.27 1.27)
+				)
+				(hide yes)
+			)
+		)
+		(property "ARTIKELKOD" "-"
 			(at 128.27 101.6 0)
 			(effects
@@
 			)
 		)
+		(property "ARTIKELKOD" "035-00209"
+			(at 182.88 73.66 0)
+			(effects
+				(font
+					(size 1.27 1.27)
+				)
+				(hide yes)
+			)
+		)
 		(pin "1"
 		)
@@
 			)
 		)
+		(property "ARTIKELKOD" "065-00195"
+			(at 146.05 63.5 0)
+			(effects
+				(font
+					(size 1.27 1.27)
+				)
+				(hide yes)
+			)
+		)
 		(pin "2"
 		)
@@
 			)
 		)
-		(property "MFR" ""
+		(property "MFR" "Omron Electronics Inc-EMC Div"
 			(at 193.04 73.66 0)
 			(effects
@@
 			)
 		)
-		(property "part-num" ""
+		(property "part-num" "B3U-1000P"
+			(at 193.04 73.66 0)
+			(effects
+				(font
+					(size 1.27 1.27)
+				)
+				(hide yes)
+			)
+		)
+		(property "ARTIKELKOD" "-"
 			(at 193.04 73.66 0)
 			(effects
@@
 			)
 		)
+		(property "ARTIKELKOD" "065-00248"
+			(at 134.62 63.5 0)
+			(effects
+				(font
+					(size 1.27 1.27)
+				)
+				(hide yes)
+			)
+		)
 		(pin "2"
 		)
@@
 			)
 		)
-		(property "Datasheet" "http://infocenter.arm.com/help/topic/com.arm.doc.ddi0314h/DDI0314H_coresight_components_trm.pdf"
+		(property "Datasheet" "~"
 			(at 193.04 133.35 90)
 			(effects
@@
 		)
 		(property "part-num" ""
+			(at 184.15 101.6 0)
+			(effects
+				(font
+					(size 1.27 1.27)
+				)
+				(hide yes)
+			)
+		)
+		(property "ARTIKELKOD" "?"
 			(at 184.15 101.6 0)
 			(effects
@@
 			)
 		)
+		(property "ARTIKELKOD" "035-00451 (15k)"
+			(at 171.45 69.85 0)
+			(effects
+				(font
+					(size 1.27 1.27)
+				)
+				(hide yes)
+			)
+		)
 		(pin "1"
 		)
@@
 			)
 		)
+		(property "ARTIKELKOD" "065-00248"
+			(at 171.45 76.2 0)
+			(effects
+				(font
+					(size 1.27 1.27)
+				)
+				(hide yes)
+			)
+		)
 		(pin "2"
 		)
@@
 			)
 		)
-		(property "MFR" ""
+		(property "MFR" "Omron Electronics Inc-EMC Div"
 			(at 85.09 100.33 0)
 			(effects
@@
 			)
 		)
-		(property "part-num" ""
+		(property "part-num" "B3U-1000P"
 			(at 85.09 100.33 0)
 			(effects
+				(font
+					(size 1.27 1.27)
+				)
+				(hide yes)
+			)
+		)
+		(property "ARTIKELKOD" "-"
+			(at 85.09 100.33 0)
+			(effects
