File: controller/hb-card.kicad_sch (KiCad schematic)
At the start: 21 parts, among them J4 Conn_01x14

Commit message: controller - Update BOM
Parts:
- C37, R112, R113, R79, R80: now not fitted
- C48: value 10nF 9V -> 100nF 9V; ARTIKELKOD (none) -> 065-00248
- C53, C58: value 1nF 100VDC -> 10nF 100VDC; ARTIKELKOD (none) -> 065-00284
- D7, D8: ARTIKELKOD (none) -> 071-00178
- J4: ARTIKELKOD (none) -> 1.5st 081-00363
- R130: value 1k -> 100R; ARTIKELKOD (none) -> 035-00440
- R17: ARTIKELKOD (none) -> 035-00450
- R18, R23, R24, R42, R43, R44, R45, R46: value ?R -> 100k; ARTIKELKOD (none) -> 035-00040; now not fitted
Changed lines of the file:
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@@
 		(in_bom yes)
 		(on_board yes)
-		(dnp no)
+		(dnp yes)
 		(property "Reference" "R80"
 			(at 72.898 53.34 90)
@@
 		(in_bom yes)
 		(on_board yes)
-		(dnp no)
+		(dnp yes)
 		(property "Reference" "R44"
 			(at 72.644 90.17 90)
@@
 			)
 		)
-		(property "Value" "?R"
+		(property "Value" "100k"
 			(at 78.74 90.17 90)
 			(effects
@@
 			)
 		)
+		(property "ARTIKELKOD" "035-00040"
+			(at 77.47 90.17 0)
+			(effects
+				(font
+					(size 1.27 1.27)
+				)
+				(hide yes)
+			)
+		)
 		(pin "2"
 		)
@@
 		(in_bom yes)
 		(on_board yes)
-		(dnp no)
+		(dnp yes)
 		(property "Reference" "R113"
 			(at 72.898 104.14 90)
@@
 		(in_bom yes)
 		(on_board yes)
-		(dnp no)
+		(dnp yes)
 		(property "Reference" "R46"
 			(at 78.486 97.282 90)
@@
 			)
 		)
-		(property "Value" "?R"
+		(property "Value" "100k"
 			(at 78.74 95.25 90)
 			(effects
@@
 			)
 		)
+		(property "ARTIKELKOD" "035-00040"
+			(at 77.47 95.25 0)
+			(effects
+				(font
+					(size 1.27 1.27)
+				)
+				(hide yes)
+			)
+		)
 		(pin "2"
 		)
@@
 		(in_bom yes)
 		(on_board yes)
-		(dnp no)
+		(dnp yes)
 		(property "Reference" "R42"
 			(at 79.502 69.596 90)
@@
 			)
 		)
-		(property "Value" "?R"
+		(property "Value" "100k"
 			(at 78.74 67.31 90)
 			(effects
@@
 			)
 		)
+		(property "ARTIKELKOD" "035-00040"
+			(at 77.47 67.31 0)
+			(effects
+				(font
+					(size 1.27 1.27)
+				)
+				(hide yes)
+			)
+		)
 		(pin "2"
 		)
@@
 			)
 		)
+		(property "ARTIKELKOD" "071-00178"
+			(at 50.8 57.15 0)
+			(effects
+				(font
+					(size 1.27 1.27)
+				)
+				(hide yes)
+			)
+		)
 		(pin "1"
 		)
@@
 			)
 		)
+		(property "ARTIKELKOD" "1.5st 081-00363"
+			(at 35.56 76.2 0)
+			(effects
+				(font
+					(size 1.27 1.27)
+				)
+				(hide yes)
+			)
+		)
 		(pin "9"
 		)
@@
 		(in_bom yes)
 		(on_board yes)
-		(dnp no)
+		(dnp yes)
 		(property "Reference" "R18"
 			(at 78.74 57.658 90)
@@
 			)
 		)
-		(property "Value" "?R"
+		(property "Value" "100k"
 			(at 78.74 59.69 90)
 			(effects
@@
 			)
 		)
+		(property "ARTIKELKOD" "035-00040"
+			(at 77.47 59.69 0)
+			(effects
+				(font
+					(size 1.27 1.27)
+				)
+				(hide yes)
+			)
+		)
 		(pin "2"
 		)
@@
 			)
 		)
-		(property "Value" "1nF 100VDC"
+		(property "Value" "10nF 100VDC"
 			(at 72.898 69.596 0)
 			(effects
@@
 			)
 		)
+		(property "ARTIKELKOD" "065-00284"
+			(at 64.77 63.5 0)
+			(effects
+				(font
+					(size 1.27 1.27)
+				)
+				(hide yes)
+			)
+		)
 		(pin "2"
 		)
@@
 		(in_bom yes)
 		(on_board yes)
-		(dnp no)
+		(dnp yes)
 		(property "Reference" "R23"
 			(at 72.898 62.23 90)
@@
 			)
 		)
-		(property "Value" "?R"
+		(property "Value" "100k"
 			(at 78.74 62.23 90)
 			(effects
@@
 			)
 		)
+		(property "ARTIKELKOD" "035-00040"
+			(at 77.47 62.23 0)
+			(effects
+				(font
+					(size 1.27 1.27)
+				)
+				(hide yes)
+			)
+		)
 		(pin "2"
 		)
@@
 		(in_bom yes)
 		(on_board yes)
-		(dnp no)
+		(dnp yes)
 		(property "Reference" "R112"
 			(at 72.898 101.6 90)
@@
 		(dnp no)
 		(property "Reference" "R130"
-			(at 126.492 81.28 90)
+			(at 131.826 80.01 0)
 			(effects
 				(font
@@
 			)
 		)
-		(property "Value" "1k"
-			(at 128.27 81.534 90)
+		(property "Value" "100R"
+			(at 131.826 81.788 0)
 			(effects
 				(font
@@
 			)
 		)
+		(property "ARTIKELKOD" "035-00440"
+			(at 128.27 81.28 0)
+			(effects
+				(font
+					(size 1.27 1.27)
+				)
+				(hide yes)
+			)
+		)
 		(pin "1"
 		)
@@
 		(in_bom yes)
 		(on_board yes)
-		(dnp no)
+		(dnp yes)
 		(property "Reference" "C37"
 			(at 125.73 86.868 0)
@@
 			)
 		)
+		(property "ARTIKELKOD" "071-00178"
+			(at 52.07 93.98 0)
+			(effects
+				(font
+					(size 1.27 1.27)
+				)
+				(hide yes)
+			)
+		)
 		(pin "1"
 		)
@@
 		(in_bom yes)
 		(on_board yes)
-		(dnp no)
+		(dnp yes)
 		(property "Reference" "R45"
 			(at 72.898 91.948 90)
@@
 			)
 		)
-		(property "Value" "?R"
+		(property "Value" "100k"
 			(at 78.74 92.71 90)
 			(effects
@@
 			)
 		)
+		(property "ARTIKELKOD" "035-00040"
+			(at 77.47 92.71 0)
+			(effects
+				(font
+					(size 1.27 1.27)
+				)
+				(hide yes)
+			)
+		)
 		(pin "2"
 		)
@@
 		(in_bom yes)
 		(on_board yes)
-		(dnp no)
+		(dnp yes)
 		(property "Reference" "R79"
 			(at 72.644 50.8 90)
@@
 			)
 		)
-		(property "Value" "1nF 100VDC"
+		(property "Value" "10nF 100VDC"
 			(at 71.628 106.426 0)
 			(effects
@@
 			)
 		)
+		(property "ARTIKELKOD" "065-00284"
+			(at 63.5 100.33 0)
+			(effects
+				(font
+					(size 1.27 1.27)
+				)
+				(hide yes)
+			)
+		)
 		(pin "2"
 		)
@@
 		(in_bom yes)
 		(on_board yes)
-		(dnp no)
+		(dnp yes)
 		(property "Reference" "R43"
 			(at 78.74 85.598 90)
@@
 			)
 		)
-		(property "Value" "?R"
+		(property "Value" "100k"
 			(at 78.74 87.63 90)
 			(effects
@@
 			)
 		)
+		(property "ARTIKELKOD" "035-00040"
+			(at 77.47 87.63 0)
+			(effects
+				(font
+					(size 1.27 1.27)
+				)
+				(hide yes)
+			)
+		)
 		(pin "2"
 		)
@@
 			)
 		)
+		(property "ARTIKELKOD" "035-00450"
+			(at 52.07 73.66 0)
+			(effects
+				(font
+					(size 1.27 1.27)
+				)
+				(hide yes)
+			)
+		)
 		(pin "2"
 		)
@@
 		(in_bom yes)
 		(on_board yes)
-		(dnp no)
+		(dnp yes)
 		(property "Reference" "R24"
 			(at 73.66 64.77 90)
@@
 			)
 		)
-		(property "Value" "?R"
+		(property "Value" "100k"
 			(at 78.74 64.77 90)
 			(effects
@@
 			)
 		)
+		(property "ARTIKELKOD" "035-00040"
+			(at 77.47 64.77 0)
+			(effects
+				(font
+					(size 1.27 1.27)
+				)
+				(hide yes)
+			)
+		)
 		(pin "2"
 		)
@@
 			)
 		)
-		(property "Value" "10nF 9V"
+		(property "Value" "100nF 9V"
 			(at 35.052 114.554 0)
 			(effects
@@
 			(at 31.75 105.41 0)
 			(effects
+				(font
+					(size 1.27 1.27)
+				)
+				(hide yes)
+			)
+		)
+		(property "ARTIKELKOD" "065-00248"
+			(at 31.75 105.41 0)
+			(effects
